Commit message: fix(description): correct timeout ownership and sensor mesh frames (#9)

File: src/mobile_base_description/urdf/mobile_base.urdf.xacro (robot description, xacro)
@@ -1,9 +1,9 @@
 <?xml version="1.0"?>
 <robot xmlns:xacro="http://www.ros.org/wiki/xacro" name="mobile_base">
-  <!-- Arguments for ros2_control configuration -->
+  <!-- Arguments for ros2_control configuration (no implicit default for timeout) -->
   <xacro:arg name="use_mock_hardware" default="false"/>
   <xacro:arg name="serial_port" default="/dev/ttyUSB0"/>
   <xacro:arg name="baud_rate" default="230400"/>
-  <xacro:arg name="response_timeout_ms" default="50"/>
+  <xacro:arg name="response_timeout_ms" default=""/>
   <!-- Include Sub-Macros -->
   <xacro:include filename="$(find mobile_base_description)/urdf/mobile_base_geometry.xacro"/>

File: src/mobile_base_description/urdf/mobile_base_geometry.xacro (robot description, xacro)
@@ -143,5 +143,6 @@
       </inertial>
       <visual>
-        <origin xyz="0 0 0" rpy="0 0 0"/>
+        <!-- Compensation RPY for CAD-oriented mesh: R_comp = inv(R_joint) -->
+        <origin xyz="0 0 0" rpy="${lidar_fl_roll} ${lidar_fl_pitch} ${lidar_fl_yaw}"/>
         <geometry>
           <mesh filename="package://mobile_base_description/meshes/base_lidar_link_FL.STL"/>
@@ -152,5 +153,5 @@
       </visual>
       <collision>
-        <origin xyz="0 0 0" rpy="0 0 0"/>
+        <origin xyz="0 0 0" rpy="${lidar_fl_roll} ${lidar_fl_pitch} ${lidar_fl_yaw}"/>
         <geometry>
           <mesh filename="package://mobile_base_description/meshes/base_lidar_link_FL.STL"/>
@@ -173,5 +174,6 @@
       </inertial>
       <visual>
-        <origin xyz="0 0 0" rpy="0 0 0"/>
+        <!-- Compensation RPY for CAD-oriented mesh: R_comp = inv(R_joint) -->
+        <origin xyz="0 0 0" rpy="${lidar_br_roll} ${lidar_br_pitch} ${lidar_br_yaw}"/>
         <geometry>
           <mesh filename="package://mobile_base_description/meshes/base_lidar_link_BR.STL"/>
@@ -182,5 +184,5 @@
       </visual>
       <collision>
-        <origin xyz="0 0 0" rpy="0 0 0"/>
+        <origin xyz="0 0 0" rpy="${lidar_br_roll} ${lidar_br_pitch} ${lidar_br_yaw}"/>
         <geometry>
           <mesh filename="package://mobile_base_description/meshes/base_lidar_link_BR.STL"/>
@@ -203,5 +205,6 @@
       </inertial>
       <visual>
-        <origin xyz="0 0 0" rpy="0 0 0"/>
+        <!-- Compensation RPY for CAD-oriented mesh: R_comp = inv(R_joint) -->
+        <origin xyz="0 0 0" rpy="0 0 ${-imu_yaw}"/>
         <geometry>
           <mesh filename="package://mobile_base_description/meshes/base_imu_link.STL"/>
@@ -212,5 +215,5 @@
       </visual>
       <collision>
-        <origin xyz="0 0 0" rpy="0 0 0"/>
+        <origin xyz="0 0 0" rpy="0 0 ${-imu_yaw}"/>
         <geometry>
           <mesh filename="package://mobile_base_description/meshes/base_imu_link.STL"/>

File: src/mobile_base_description/urdf/mobile_base_ros2_control.xacro (robot description, xacro)
@@ -5,5 +5,5 @@
     serial_port:=/dev/ttyUSB0
     baud_rate:=230400
-    response_timeout_ms:=50
+    response_timeout_ms:=''
     left_driver_id:=2
     right_driver_id:=1
@@ -18,5 +18,7 @@
         <param name="serial_port">${serial_port}</param>
         <param name="baud_rate">${baud_rate}</param>
-        <param name="response_timeout_ms">${response_timeout_ms}</param>
+        <xacro:if value="${response_timeout_ms != ''}">
+          <param name="response_timeout_ms">${response_timeout_ms}</param>
+        </xacro:if>
         <param name="left_driver_id">${left_driver_id}</param>
         <param name="right_driver_id">${right_driver_id}</param>
