Commit message: Record verified sensor mounting and reconcile model launch (#37 #38)

File: reference/FIH_AMR_ROBOT_V2.0_0731/urdf/RWF_V2.0_QA_release.urdf (robot description, URDF)
Before this commit: robot RWF_V2_0702, 85 links, 84 joints
Joints:
- joint base_imu_joint: origin xyz=0.0437499999999998 -0.00799999999999978 -0.0145899999999999 rpy=0 0 0 -> xyz=0.0437499999999998 -0.00799999999999978 -0.0145899999999999 rpy=0 0 1.5707963267948966
- joint base_lidar_joint_BR: origin xyz=-0.24671 -0.26721 -0.06011 rpy=0 0 0 -> xyz=-0.24671 -0.26721 -0.06011 rpy=3.141592653589793 0 -2.356194490192345
- joint base_lidar_joint_FL: origin xyz=0.28771 0.26721 -0.06011 rpy=0 0 0 -> xyz=0.28771 0.26721 -0.06011 rpy=3.141592653589793 0 0.7853981633974483
